Commit message: fix wheel, keyboard control, and model to predict both steering angle and velocity

File: src/drivex_description/urdf/drivex_ackermann.urdf.xacro (robot description, xacro)
@@ -2,19 +2,20 @@
 <robot name="drivex" xmlns:xacro="http://www.ros.org/wiki/xacro">
     <!--
-    Robot model taken from http://wiki.ros.org/pr2_mechanism/Tutorials/SImple%20URDF-Controller%20Example
+    Robot model taken from
+    http://wiki.ros.org/pr2_mechanism/Tutorials/SImple%20URDF-Controller%20Example
     -->
-    <xacro:include filename="$(find drivex_description)/urdf/drivex_wheel.urdf.xacro"/>
-    <xacro:include filename="$(find drivex_description)/urdf/drivex_ackermann_macro.urdf.xacro"/>
-    <xacro:include filename="$(find drivex_description)/urdf/sensors_macro.urdf.xacro"/>
-    <xacro:property name="deg_to_rad" value="0.01745329251994329577"/>
+    <xacro:include filename="$(find drivex_description)/urdf/drivex_wheel.urdf.xacro" />
+    <xacro:include filename="$(find drivex_description)/urdf/drivex_ackermann_macro.urdf.xacro" />
+    <xacro:include filename="$(find drivex_description)/urdf/sensors_macro.urdf.xacro" />
+    <xacro:property name="deg_to_rad" value="0.01745329251994329577" />
     <!-- Constants for robot dimensions -->
     <xacro:property name="length" value="0.6" />  <!-- Length between front & rear wheels -->
     <xacro:property name="width" value="0.2" /> <!-- width between left & right wheels -->
-    <xacro:property name="height" value="0.5"/>
-    <xacro:property name="length_offset" value="0"/>
-    <xacro:property name="height_offset" value="0"/>
-    <xacro:property name="wheel_radius" value="0.06" /> <!-- Link 1 -->
-    <xacro:property name="board_height" value="0.15" /> <!-- Link 1 -->
-    <xacro:property name="thickness" value="0.032" /> <!-- Link 2 -->
+    <xacro:property name="height" value="0.5" />
+    <xacro:property name="length_offset" value="0" />
+    <xacro:property name="height_offset" value="0" />
+    <xacro:property name="wheel_radius" value="0.033" />
+    <xacro:property name="wheel_thickness" value="0.028" />
+    <xacro:property name="board_height" value="0.15" />
     <!--  we need two because the car isn't a square-->
     <xacro:property name="axel_offset_x" value="0.5" /> <!-- Space btw top of beam and the each joint -->
@@ -22,32 +23,47 @@
     <xacro:property name="steer_offset" value="0.02" /> <!-- Link 1 -->
     <!-- Add car macro -->
-    <xacro:drivex length="${length}" width="${width}" height="${height}" board_height="${board_height}" wheel_radius="${wheel_radius}"/>
+    <xacro:drivex length="${length}" width="${width}" height="${height}"
+        board_height="${board_height}" wheel_radius="${wheel_radius}" />
     <!-- Add sensors-->
-    <!-- <xacro:kinect name="top_front_camera" x= "-0.22" y="0" z="0.6" roll="0" pitch="0.4" yaw="0"/> -->
-    <xacro:usb_cam name="bottom_front_camera" x="0.1" y="0" z="0.6" roll="0" pitch="0.6" yaw="0"/>
+    <!-- <xacro:kinect name="top_front_camera" x= "-0.22" y="0" z="0.6" roll="0" pitch="0.4"
+    yaw="0"/> -->
+    <xacro:usb_cam name="bottom_front_camera" x="0.1" y="0" z="0.18" roll="0" pitch="0.5" yaw="0" />
     <!-- Add gazebo functionalities-->
-    <xacro:include filename="$(find drivex_description)/urdf/drivex.gazebo.macro.xacro"/>
+    <xacro:include filename="$(find drivex_description)/urdf/drivex.gazebo.macro.xacro" />
     <!-- joints for ackermann_steering_controller -->
-    <xacro:front_steer name="front" parent="base" radius="${wheel_radius}" thickness="${thickness}"
-                       length="${length}" width="${width}" axel_offset="${axel_offset_x}" steer_height="${wheel_radius+steer_offset}">
-        <origin xyz="${length/2-axel_offset_x} 0 0" rpy="${-90 * deg_to_rad} 0 ${90 * deg_to_rad}"/>
+    <xacro:front_steer name="front" parent="base" radius="${wheel_radius}"
+        thickness="${wheel_thickness}"
+        length="${length}" width="${width}" axel_offset="${axel_offset_x}"
+        steer_height="${wheel_radius+steer_offset}">
+        <origin xyz="${length/2-axel_offset_x} 0 0" rpy="${-90 * deg_to_rad} 0 ${90 * deg_to_rad}" />
     </xacro:front_steer>
-    <xacro:rear_wheel name="rear" parent="base" radius="${wheel_radius}" thickness="${thickness}">
-        <origin xyz="${-length/2+axel_offset_x} 0 0" rpy="${-90 * deg_to_rad} 0 ${-90 * deg_to_rad}"/>
+    <xacro:rear_wheel name="rear" parent="base" radius="${wheel_radius}"
+        thickness="${wheel_thickness}">
+        <origin xyz="${-length/2+axel_offset_x} 0 0" rpy="${-90 * deg_to_rad} 0 ${-90 * deg_to_rad}" />
     </xacro:rear_wheel>
     <!-- Wheels (Keep!!) -->
-    <xacro:front_wheel_lr name="front_right" parent="base" radius="${wheel_radius}" thickness="${thickness}"
-                          length="${2*length + 0.1}" width="${width}" axel_offset="${axel_offset_x}" right_left="1" steer_height="${wheel_radius+steer_offset}">
-        <origin xyz="${length/2-axel_offset_x + 0.05} ${width/2+axel_offset_y} 0" rpy="${-90 * deg_to_rad} 0 0"/>
+    <xacro:front_wheel_lr name="front_right" parent="base" radius="${wheel_radius}"
+        thickness="${wheel_thickness}"
+        length="${2*length + 0.07}" width="${width}" axel_offset="${axel_offset_x}" right_left="1"
+        steer_height="${wheel_radius+steer_offset}">
+        <origin xyz="${length/2-axel_offset_x} ${width/2+axel_offset_y} 0"
+            rpy="${-90 * deg_to_rad} 0 0" />
     </xacro:front_wheel_lr>
-    <xacro:front_wheel_lr name="front_left" parent="base" radius="${wheel_radius}" thickness="${thickness}"
-                          length="${2*length + 0.1}" width="${width}" axel_offset="${axel_offset_x}" right_left="-1" steer_height="${wheel_radius+steer_offset}">
-        <origin xyz="${length/2-axel_offset_x + 0.05} ${-width/2-axel_offset_y} 0" rpy="${-90 * deg_to_rad} 0 0"/>
+    <xacro:front_wheel_lr name="front_left" parent="base" radius="${wheel_radius}"
+        thickness="${wheel_thickness}"
+        length="${2*length + 0.07}" width="${width}" axel_offset="${axel_offset_x}" right_left="-1"
+        steer_height="${wheel_radius+steer_offset}">
+        <origin xyz="${length/2-axel_offset_x} ${-width/2-axel_offset_y} 0"
+            rpy="${-90 * deg_to_rad} 0 0" />
     </xacro:front_wheel_lr>
-    <xacro:rear_wheel_lr name="rear_right" parent="base" radius="${wheel_radius}" right_left="1" thickness="${thickness}">
-        <origin xyz="${length/2-axel_offset_x + 0.05} ${width/2+axel_offset_y} 0" rpy="${-90 * deg_to_rad} 0 ${-90 * deg_to_rad}"/>
+    <xacro:rear_wheel_lr name="rear_right" parent="base" radius="${wheel_radius}" right_left="1"
+        thickness="${wheel_thickness}">
+        <origin xyz="${length/2-axel_offset_x + 0.065} ${width/2+axel_offset_y} 0"
+            rpy="${-90 * deg_to_rad} 0 ${-90 * deg_to_rad}" />
     </xacro:rear_wheel_lr>
-    <xacro:rear_wheel_lr name="rear_left" parent="base" radius="${wheel_radius}" right_left="-1" thickness="${thickness}">
-        <origin xyz="${length/2-axel_offset_x + 0.05} ${-width/2-axel_offset_y} 0" rpy="${-90 * deg_to_rad} 0 ${90 * deg_to_rad}"/>
+    <xacro:rear_wheel_lr name="rear_left" parent="base" radius="${wheel_radius}" right_left="-1"
+        thickness="${wheel_thickness}">
+        <origin xyz="${length/2-axel_offset_x + 0.065} ${-width/2-axel_offset_y} 0"
+            rpy="${-90 * deg_to_rad} 0 ${90 * deg_to_rad}" />
     </xacro:rear_wheel_lr>
     <!-- Gazebo plugin for ROS Control -->

File: src/drivex_description/urdf/drivex_ackermann_macro.urdf.xacro (robot description, xacro)
@@ -32,5 +32,5 @@
                 <origin xyz="0 0 -0.05" rpy="0 0 0"/>
                 <geometry>
-                    <mesh filename="file:///$(find drivex_description)/meshes/chassis_bfmc.dae" scale="1 1 1"/>
+                    <mesh filename="file:///$(find drivex_description)/meshes/chassis.dae" scale="1 1 1"/>
                 </geometry>
                 <material name="material">
@@ -69,5 +69,5 @@
                 <origin xyz="0 0 -0.06" rpy="0 0 0"/>
                 <geometry>
-                    <mesh filename="file:///$(find drivex_description)/meshes/CarBody_bfmc.dae" scale="1 1 1"/>
+                    <mesh filename="file:///$(find drivex_description)/meshes/CarBody.dae" scale="1 1 1"/>
                 </geometry>
                 <material name="CarBody">
